Commit message: Easier (laserscan friendly) collisions for the table

File: urdf/table.urdf.xacro (robot description, xacro)
@@ -1,4 +1,5 @@
 <?xml version="1.0"?>
 <robot name="table" xmlns:xacro="http://ros.org/wiki/xacro">
+    <xacro:arg name="easy_collision" default="false"/>
     <material name="table_colour">
         <color rgba="0.1 0.1 0.4 1"/>
@@ -22,8 +23,16 @@
         </visual>
         <collision>
-            <origin xyz="0 0 0" rpy="0 0 0" />
-            <geometry>
-                <box size="2.74 1.525 0.03" />
-            </geometry>
+            <xacro:if value="$(arg easy_collision)">
+                <origin xyz="0 0 -0.37" rpy="0 0 0" />
+                <geometry>
+                    <box size="2.74 1.525 0.74" />
+                </geometry>
+            </xacro:if>
+            <xacro:unless value="$(arg easy_collision)">
+                <origin xyz="0 0 0" rpy="0 0 0" />
+                <geometry>
+                    <box size="2.74 1.525 0.03" />
+                </geometry>
+            </xacro:unless>
         </collision>
     </link>
@@ -136,8 +145,16 @@
         </visual>
         <collision>
-            <origin xyz="0 0 0" rpy="0 0 0" />
-            <geometry>
-                <box size="0.002 1.83 0.1525" />
-            </geometry>
+            <xacro:if value="$(arg easy_collision)">
+                <origin xyz="0 0 -0.37" rpy="0 0 0" />
+                <geometry>
+                    <box size="0.002 1.83 0.8925" />
+                </geometry>
+            </xacro:if>
+            <xacro:unless value="$(arg easy_collision)">
+                <origin xyz="0 0 0" rpy="0 0 0" />
+                <geometry>
+                    <box size="0.002 1.83 0.1525" />
+                </geometry>
+            </xacro:unless>
         </collision>
     </link>

Commit message: Increased the collision of the table when using the easy collision arg

File: urdf/table.urdf.xacro (robot description, xacro)
@@ -26,5 +26,5 @@
                 <origin xyz="0 0 -0.37" rpy="0 0 0" />
                 <geometry>
-                    <box size="2.74 1.525 0.74" />
+                    <box size="2.74 1.525 0.77" />
                 </geometry>
             </xacro:if>
